File: Sous_Vide/Sous_Vide.sch (KiCad schematic (older format))
At the start: 5 parts

Commit message: something
Parts:
- removed IC?: ATTINY85-S, SO8-200, symbol ATTINY85-S
- added IC?: ATTINY85-S, SO8-200, symbol ATTINY85-S-RESCUE-Sous_Vide
- added P?: CONN_02X03, symbol CONN_02X03
- added R? (x2): R, symbol R
- added SW? (x2): SW_PUSH, symbol SW_PUSH
Connections:
- net labels added: +5V, CTRL, MISO, MOSI, RST, SCK
- wire segments 0 -> 22
Other:
- moved on the sheet: K?, R?, SW?
