File: Patriot_Companion_Simplified/Patriot_Companion.kicad_pcb (KiCad board)
At the start: 2 copper layers, 82 parts, among them P1 USB_OTG, P2 POWER_IN, P3 I/O, P4 CONN_02X03, P5 MOTOR_1, P6 MOTOR_2, P7 SERVO_HEADER, Q1 FDN340P, SW1 SWITCH, SW2 SWITCH, SW3 SWITCH, U1 LM358, U2 ATMEGA32U4-A, U3 LP2985-33DBVR, U4 7805, U5 BD6212HFP-TR, U6 NXP_MMA8652FCR1, U7 BD6212HFP-TR, U8 Si7006, Y1 16M

Commit message: update
Parts:
- removed C17: 1u0, Capacitors_SMD:C_0603_HandSoldering
- removed C18, C19, C22: 0u1, Capacitors_SMD:C_0603_HandSoldering
- removed RV3: POT_Dual_Separate, DM_Custom:IM_joystick
- removed U6: NXP_MMA8652FCR1, DM_Custom:NXP_MMA8652FCR1_hand
- added G***: LOGO, KiCad_Footprints:ZF_LOGO_PHHS, B.Cu at (294.4, 125.0)
- added G***: LOGO, KiCad_Footprints:ZF_LOGO_MPS, F.Cu at (233.3, 104.1)
- added REF**: ZF_STRUCT_M3-hole, KiCad_Footprints:ZF_STRUCT_M3-hole, F.Cu at (267.5, 100.0)
- added REF**: ZF_STRUCT_M3-hole, KiCad_Footprints:ZF_STRUCT_M3-hole, F.Cu at (267.5, 125.0)
- added REF**: ZF_STRUCT_M3-hole, KiCad_Footprints:ZF_STRUCT_M3-hole, F.Cu at (202.5, 125.0)
- added REF**: ZF_STRUCT_M3-hole, KiCad_Footprints:ZF_STRUCT_M3-hole, F.Cu at (202.5, 100.0)
- added U9: joystick, KiCad_Footprints:ZF_JOYSTICK, F.Cu at (219.0, 112.5)
- 1u1, C10, C11, C12, C13, C15, C16, C20, C24, C3, C4, C5, C6, C7, C8, C9, F1, L1, L2, Q1, R1, R11, R12, R15, R16, R2, R4, RV1, RV2, U1, U3: moved to B.Cu
- C21, C25: footprint Capacitors_SMD:C_0603_HandSoldering -> KiCad_Footprints:ZF_SMD_pol_1206; moved to B.Cu
- D2: footprint Diodes_SMD:D_SOT-23_ANK -> KiCad_Footprints:ZF_SMD_pol_0805; moved to B.Cu
- P1: footprint Connectors:USB_Micro-B -> KiCad_Footprints:ZF_CONN_USB-MICRO-B-SMD-holes
- P2: footprint Connectors:BARREL_JACK -> KiCad_Footprints:ZF_CONN_POWER_1x2
- P3: value I/O -> CONN_01X07; footprint Pin_Headers:Pin_Header_Angled_1x04_Pitch1.27mm -> KiCad_Footprints:ZF_CONN_1x7-hdr
- P4: footprint Pin_Headers:Pin_Header_Angled_2x03_Pitch1.27mm -> KiCad_Footprints:ZF_CONN_3x2_noshroud
- P5, P6: footprint Connectors_Terminal_Blocks:TerminalBlock_Pheonix_PT-3.5mm_2pol -> KiCad_Footprints:ZF_CONN_POWER_1x2
- P7: footprint Pin_Headers:Pin_Header_Angled_1x03_Pitch1.27mm -> KiCad_Footprints:ZF_CONN_1x3_servo
- R13, R14: value 1k -> R; footprint Resistors_SMD:R_0603_HandSoldering -> KiCad_Footprints:ZF_SMD_NonPol_0603
- SW1: footprint DM_Custom:DM_CUSTOM_B3FS-4 -> KiCad_Footprints:ZF_SW_LS38
- U2: footprint DM_Custom:LW_CUSTOM_ATMEGA32 -> KiCad_Footprints:ZF_IC_TQFP44-0-8
- U4: value 7805 -> LF33CDT-TRY; footprint DM_Custom:AZ_Custom_Mosfet -> KiCad_Footprints:ZF_SMD_DPAK; moved to B.Cu
- moved C23 166.1 mm to (253.8, 92.8)
- moved U3 153.0 mm to (231.9, 112.0)
- moved 1u1 152.0 mm to (229.7, 112.0), turned to 270 degrees
- moved Q1 150.3 mm to (235.0, 113.0), turned to 270 degrees
- moved LED5 150.3 mm to (257.7, 169.0)
- moved LED8 150.3 mm to (256.2, 150.8)
- moved LED1 150.3 mm to (245.0, 151.0)
- moved LED2 150.3 mm to (238.7, 156.6)
- moved LED3 150.3 mm to (238.7, 163.2)
- moved LED4 150.3 mm to (264.1, 163.2)
- moved LED6 150.3 mm to (245.3, 169.0)
- moved LED7 150.3 mm to (264.1, 156.6)
- moved R2 147.7 mm to (230.5, 96.5)
- moved C13 145.2 mm to (240.2, 119.8), turned to 180 degrees
- moved C11 144.1 mm to (231.9, 114.9), turned to 180 degrees
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Connections:
- R13 pad 1: +3V3 -> D-
- R13 pad 2: SCL -> Net-(P1-Pad2)
- R14 pad 1: +3V3 -> D+
- R14 pad 2: SDA -> Net-(P1-Pad3)
- U2 pad 1: Net-(U2-Pad1) -> Net-(P3-Pad1)
- U2 pad 12: ACCEL_INT -> Net-(U2-Pad12)
- U2 pad 38: Net-(P3-Pad4) -> Net-(P3-Pad5)
- U2 pad 39: Net-(P3-Pad3) -> Net-(P3-Pad4)
- U2 pad 40: Net-(P3-Pad2) -> Net-(P3-Pad3)
- U2 pad 41: Net-(P3-Pad1) -> Net-(P3-Pad2)
- U4 pad 1: (no net) -> VSS
- U4 pad 2: (no net) -> GND
- U4 pad 3: (no net) -> +5V
Routing:
- net (no net): track 0.00 -> 76.5 mm
- net Net-(P6-Pad1): track 43.1 -> 0.00 mm, vias 1 -> 0
- net VUSB: track 0.00 -> 38.1 mm, vias 0 -> 1
- net Net-(P6-Pad2): track 37.1 -> 0.00 mm, vias 1 -> 0
- net RIN1: track 29.6 -> 0.04 mm
- net FIN1: track 27.8 -> 0.00 mm
- net FIN2: track 30.3 -> 3.64 mm, vias 0 -> 1
- net RIN2: track 30.2 -> 3.74 mm, vias 0 -> 1
- net Net-(P5-Pad1): track 24.0 -> 0.00 mm, vias 1 -> 0
- net +5V: track 43.5 -> 66.6 mm, vias 0 -> 3
- net GND: track 11.5 -> 32.1 mm, vias 0 -> 6
- net SDA: track 0.00 -> 19.9 mm
- net Net-(C12-Pad1): track 0.00 -> 19.5 mm, vias 0 -> 2
- net Net-(R7-Pad2): track 0.00 -> 19.3 mm, vias 0 -> 2
- net SCL: track 0.00 -> 19.2 mm
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- added copper zone on B.Cu, net GND
Other:
- board outline added: 70 x 30 mm
- net class Default: trace_width 0.25 -> 0.2
- rule pad_to_mask_clearance: 0.2 -> 0
- board text added: "PHHS"
