File: Patriot_Companion_Simplified/Patriot_Companion.sch (KiCad schematic (older format))
At the start: 82 parts, among them P1 USB_OTG, P2 POWER_IN, P3 I/O, P4 CONN_02X03, P5 MOTOR_1, P6 MOTOR_2, P7 SERVO_HEADER, Q1 FDN340P, SW1 SWITCH, SW2 SWITCH, SW3 SWITCH, U1 LM358, U2 ATMEGA32U4-A, U3 LP2985-33DBVR, U4 7805, U5 BD6212HFP-TR, U6 NXP_MMA8652FCR1, U7 BD6212HFP-TR, U8 Si7006, Y1 16M

Commit message: update
Parts:
- removed C17: 1u0, Capacitors_SMD:C_0603_HandSoldering, symbol C
- removed C18, C19, C22: 0u1, Capacitors_SMD:C_0603_HandSoldering, symbol C
- removed P3: I/O, Pin_Headers:Pin_Header_Angled_1x04_Pitch1.27mm, symbol CONN_01X04
- removed RV3: POT_Dual_Separate, DM_Custom:IM_joystick, symbol POT_Dual_Separate
- removed U4: 7805, DM_Custom:AZ_Custom_Mosfet, symbol 7805
- removed U6: NXP_MMA8652FCR1, DM_Custom:NXP_MMA8652FCR1_hand, symbol NXP_MMA8652FCR1
- added P3: CONN_01X07, KiCad_Footprints:ZF_CONN_1x7-hdr, symbol CONN_01X07
- added U4: LF33CDT-TRY, KiCad_Footprints:ZF_SMD_DPAK, symbol LF33CDT-TRY
- added U9: joystick, KiCad_Footprints:ZF_JOYSTICK, symbol joystick
- C21, C25: footprint Capacitors_SMD:C_0603_HandSoldering -> KiCad_Footprints:ZF_SMD_pol_1206; RoHS (none) -> Yes; Subs Allowed (none) -> No
- D2: footprint Diodes_SMD:D_SOT-23_ANK -> KiCad_Footprints:ZF_SMD_pol_0805; RoHS (none) -> Yes; Subs Allowed (none) -> No
- P1: footprint Connectors:USB_Micro-B -> KiCad_Footprints:ZF_CONN_USB-MICRO-B-SMD-holes
- P2: footprint Connectors:BARREL_JACK -> KiCad_Footprints:ZF_CONN_POWER_1x2; RoHS (none) -> Yes; Subs Allowed (none) -> No
- P4: footprint Pin_Headers:Pin_Header_Angled_2x03_Pitch1.27mm -> KiCad_Footprints:ZF_CONN_3x2_noshroud; RoHS (none) -> Yes; Subs Allowed (none) -> No
- P5, P6: footprint Connectors_Terminal_Blocks:TerminalBlock_Pheonix_PT-3.5mm_2pol -> KiCad_Footprints:ZF_CONN_POWER_1x2; RoHS (none) -> Yes; Subs Allowed (none) -> No
- P7: footprint Pin_Headers:Pin_Header_Angled_1x03_Pitch1.27mm -> KiCad_Footprints:ZF_CONN_1x3_servo; RoHS (none) -> Yes; Subs Allowed (none) -> No
- R13, R14: value 1k -> R; footprint Resistors_SMD:R_0603_HandSoldering -> KiCad_Footprints:ZF_SMD_NonPol_0603; RoHS (none) -> Yes; Subs Allowed (none) -> No
- SW1: footprint DM_Custom:DM_CUSTOM_B3FS-4 -> KiCad_Footprints:ZF_SW_LS38; RoHS (none) -> Yes; Subs Allowed (none) -> No
- U2: footprint DM_Custom:LW_CUSTOM_ATMEGA32 -> KiCad_Footprints:ZF_IC_TQFP44-0-8; RoHS (none) -> Yes; Subs Allowed (none) -> No
- U3: footprint DM_Custom:NB_Custom_S-L2985 -> KiCad_Footprints:ZF_SOT23-5L; RoHS (none) -> Yes; Subs Allowed (none) -> No
Connections:
- net +3V3: no longer R13.1, R14.1
- net +5V: now also U4.3 (Vout), U9.1 (L/R+), U9.8 (U/D+)
- net D+: now also R14.1
- net D-: now also R13.1
- net GND: now also U4.2 (GND), U9.4 (GND), U9.5 (GND)
- net JOYSTICK_X: now also U9.7 (L/R)
- net JOYSTICK_Y: now also U9.6 (U/D)
- net SCL: now also P3.6 (P6); no longer R13.2
- net SDA: now also P3.7 (P7); no longer R14.2
- net VSS: now also U4.1 (Vin)
- net at U2.1 ((INT6/AIN0)PE6): now also P3.1 (P1)
- net at U2.38 ((ADC5/TMS)PF5): now also P3.5 (P5)
- net at U2.39 ((ADC4/TCK)PF4): now also P3.4 (P4)
- net at U2.40 ((ADC1)PF1): now also P3.3 (P3)
- net at U2.41 ((ADC0)PF0): now also P3.2 (P2)
- net at P1.2 (D-), RV1.1: now also R13.2
- net at P1.3 (D+), RV2.1: now also R14.2
- net ACCEL_INT: no longer names the net of U2.12 ((OC0A/OC1C/~RTS~/PCINT7)PB7)
Other:
- note removed: "ACCELEROMETER"
- note removed: "I/O HEADER"
- moved on the sheet: C20, C21, C24, C25, P5, P6, R11, R12, R15, R16, U5, U7
