File: Patriot_Companion/Patriot_Companion.kicad_pcb (KiCad board)
At the start: 2 copper layers, 82 parts, among them P1 USB_OTG, P2 POWER_IN, P3 I/O, P4 CONN_02X03, P5 MOTOR_1, P6 MOTOR_2, P7 SERVO_HEADER, Q1 FDN340P, SW1 SWITCH, SW2 SWITCH, SW3 SWITCH, U1 LM358, U2 ATMEGA32U4-A, U3 LP2985-33DBVR, U4 7805, U5 BD6212HFP-TR, U6 NXP_MMA8652FCR1, U7 BD6212HFP-TR, U8 Si7006, Y1 16M

Commit message: started PC routes
Parts:
- LED1, LED2, LED3, LED4, LED5, LED6, LED7, LED8, RV3, SW2, SW3, U6: moved to B.Cu
- moved L1 178.2 mm to (81.3, 158.5), turned to 270 degrees
- moved P1 169.1 mm to (76.7, 139.2), turned to 270 degrees
- moved U3 165.7 mm to (85.3, 156.0)
- moved F1 155.2 mm to (79.5, 145.8), turned to 180 degrees
- moved D2 148.7 mm to (105.9, 158.8)
- moved C7 144.7 mm to (88.9, 140.0)
- moved C8 140.4 mm to (88.6, 143.5), turned to 180 degrees
- moved C6 139.4 mm to (88.4, 137.2)
- moved P2 138.2 mm to (120.9, 157.2), turned to 90 degrees
- moved U1 138.0 mm to (89.9, 158.0), turned to 180 degrees
- moved C11 135.8 mm to (95.2, 160.5)
- moved C4 134.4 mm to (83.3, 129.8)
- moved R7 131.3 mm to (104.9, 130.3)
- moved R2 130.8 mm to (95.5, 156.5)
- moved 1u1 130.6 mm to (83.1, 151.9)
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Routing:
- net Net-(P6-Pad1): track 0.00 -> 43.1 mm, vias 0 -> 1
- net Net-(P6-Pad2): track 0.00 -> 37.1 mm, vias 0 -> 1
- net FIN2: track 0.00 -> 30.3 mm
- net RIN2: track 0.00 -> 30.2 mm
- net RIN1: track 0.00 -> 29.6 mm
- net FIN1: track 0.00 -> 27.8 mm
- net Net-(P5-Pad1): track 0.00 -> 24.0 mm, vias 0 -> 1
- net Net-(P5-Pad2): track 0.00 -> 19.0 mm, vias 0 -> 1
- net GND: track 0.00 -> 11.5 mm
- net +5V: track 47.5 -> 43.5 mm, vias 2 -> 0

Commit message: update
Changed lines of the file:
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@@
     (links 203)
     (no_connects 183)
-    (area 34.801999 13.364999 229.409048 168.365)
+    (area 70.723 74.264 183.531001 171.451001)
     (thickness 1.6)
     (drawings 0)
-    (tracks 60)
+    (tracks 61)
     (zones 0)
     (modules 82)
@@
   (segment (start 124.31 137.838) (end 124.46 137.988) (width 0.5) (layer F.Cu) (net 2))
   (segment (start 124.46 137.988) (end 128.27 137.988) (width 0.5) (layer F.Cu) (net 2))
+  (segment (start 135.128 131.572) (end 135.128 134.874) (width 0.5) (layer F.Cu) (net 10))
+  (segment (start 135.128 128.016) (end 135.128 131.572) (width 0.5) (layer F.Cu) (net 10))
   (segment (start 132.1895 127.635) (end 134.747 127.635) (width 0.5) (layer F.Cu) (net 10))
   (segment (start 134.747 135.255) (end 132.1895 135.255) (width 0.5) (layer F.Cu) (net 10))
   (segment (start 135.128 134.874) (end 134.747 135.255) (width 0.5) (layer F.Cu) (net 10))
-  (segment (start 135.128 128.016) (end 135.128 134.874) (width 0.5) (layer F.Cu) (net 10))
   (segment (start 134.747 127.635) (end 135.128 128.016) (width 0.5) (layer F.Cu) (net 10))
   (segment (start 124.46 133.67) (end 128.27 133.67) (width 0.5) (layer F.Cu) (net 10))

Commit message: ISP done
Parts:
- removed 1u1, C23: C, Capacitors_SMD:C_0603_HandSoldering
- removed C11: 1u, Capacitors_SMD:C_0603_HandSoldering
- removed C17: 1u0, Capacitors_SMD:C_0603_HandSoldering
- removed C18, C19, C22: 0u1, Capacitors_SMD:C_0603_HandSoldering
- removed LED4, LED5, LED6, LED7, LED8: NeoPixel, DM_Custom:SR_CUSTOM_NEO_PIX
- removed Q1: FDN340P, TO_SOT_Packages_SMD:SOT-23_Handsoldering
- removed R17, R18: R, Resistors_SMD:R_0603_HandSoldering
- removed RV3: POT_Dual_Separate, DM_Custom:IM_joystick
- removed U3: LP2985-33DBVR, DM_Custom:NB_Custom_S-L2985
- removed U6: NXP_MMA8652FCR1, DM_Custom:NXP_MMA8652FCR1_hand
- removed U8: Si7006, DM_Custom:SM_Custom_Si7006
- added D5: LED, KiCad_Footprints:ZF_SMD_pol_0805, F.Cu at (234.9, 124.7)
- added D6: D, KiCad_Footprints:ZF_SMD_pol_0805, B.Cu at (233.0, 119.5)
- added F2: Polyfuse, KiCad_Footprints:ZF_SMD_1812, B.Cu at (245.8, 124.0)
- added G***: LOGO, KiCad_Footprints:ZF_LOGO_PHHS, F.Cu at (239.7, 114.0)
- added R19: R, KiCad_Footprints:ZF_SMD_NonPol_0603, B.Cu at (234.9, 126.2)
- added REF**: ZF_STRUCT_M3-hole, KiCad_Footprints:ZF_STRUCT_M3-hole, F.Cu at (267.5, 100.0)
- added REF**: ZF_STRUCT_M3-hole, KiCad_Footprints:ZF_STRUCT_M3-hole, F.Cu at (267.5, 125.0)
- added REF**: ZF_STRUCT_M3-hole, KiCad_Footprints:ZF_STRUCT_M3-hole, F.Cu at (202.5, 125.0)
- added REF**: ZF_STRUCT_M3-hole, KiCad_Footprints:ZF_STRUCT_M3-hole, F.Cu at (202.5, 100.0)
- added U9: joystick, KiCad_Footprints:ZF_JOYSTICK, F.Cu at (219.0, 112.5)
- C10: footprint Capacitors_SMD:C_0603_HandSoldering -> KiCad_Footprints:ZF_SMD_NonPol_0603; moved to B.Cu
- C12, C20, C24, C4, C5, C6, C7, C8, C9, L1, L2, R10, R11, R12, R15, R16, R4, R9, RV1, RV2: moved to B.Cu
- C13, C15, C16: footprint SMD_Packages:SMD-1206_Pol -> KiCad_Footprints:ZF_SMD_pol_1206; moved to B.Cu
- C21, C25: footprint Capacitors_SMD:C_0603_HandSoldering -> KiCad_Footprints:ZF_SMD_pol_1206; moved to B.Cu
- C3: value C -> 0u1; footprint Capacitors_SMD:C_0603_HandSoldering -> KiCad_Footprints:ZF_SMD_NonPol_0603; moved to B.Cu
- D2: footprint Diodes_SMD:D_SOT-23_ANK -> KiCad_Footprints:ZF_SMD_pol_0805; moved to B.Cu
- F1: footprint Resistors_SMD:R_1812_HandSoldering -> KiCad_Footprints:ZF_SMD_1812; moved to B.Cu
- LED1, LED2, LED3: moved to F.Cu
- P1: footprint Connectors:USB_Micro-B -> KiCad_Footprints:ZF_CONN_USB-MICRO-B-SMD-holes
- P2: footprint Connectors:BARREL_JACK -> KiCad_Footprints:ZF_CONN_POWER_1x2
- P3: value I/O -> CONN_01X07; footprint Pin_Headers:Pin_Header_Angled_1x04_Pitch1.27mm -> KiCad_Footprints:ZF_CONN_1x7-hdr
- P4: footprint Pin_Headers:Pin_Header_Angled_2x03_Pitch1.27mm -> KiCad_Footprints:ZF_CONN_3x2_noshroud
- P5, P6: footprint Connectors_Terminal_Blocks:TerminalBlock_Pheonix_PT-3.5mm_2pol -> KiCad_Footprints:ZF_CONN_POWER_1x2
- P7: footprint Pin_Headers:Pin_Header_Angled_1x03_Pitch1.27mm -> KiCad_Footprints:ZF_CONN_1x3_servo
- R1, R2: value 10k -> R; footprint Resistors_SMD:R_0603_HandSoldering -> KiCad_Footprints:ZF_SMD_NonPol_0603; moved to B.Cu
- R13, R14: value 1k -> R; footprint Resistors_SMD:R_0603_HandSoldering -> KiCad_Footprints:ZF_SMD_NonPol_0603
- SW1: footprint DM_Custom:DM_CUSTOM_B3FS-4 -> KiCad_Footprints:ZF_SW_LS38
- SW2, SW3: footprint DM_Custom:DM_CUSTOM_B3FS-4 -> KiCad_Footprints:ZF_SW_Metal_Ball_Tactile; moved to F.Cu
- U1: value LM358 -> SHT30-DIS-B; footprint DM_Custom:DM_CUSTOM_LM398_S08 -> KiCad_Footprints:ZF_IC_DFN8-050
- U2: footprint DM_Custom:LW_CUSTOM_ATMEGA32 -> KiCad_Footprints:ZF_IC_TQFP44-0-8
- U4: value 7805 -> LF33CDT-TRY; footprint DM_Custom:AZ_Custom_Mosfet -> KiCad_Footprints:ZF_SMD_DPAK; moved to B.Cu
- moved SW2 177.2 mm to (266.2, 112.5), turned to 90 degrees
- moved SW3 173.1 mm to (258.4, 112.5), turned to 90 degrees
- moved U1 157.7 mm to (237.0, 101.1)
- moved C3 154.6 mm to (247.0, 119.5), turned to 90 degrees
- moved LED3 151.4 mm to (240.0, 118.2), turned to 270 degrees
- moved R2 151.3 mm to (237.0, 102.8)
- moved R1 151.2 mm to (237.0, 99.4), turned to 0 degrees
- moved C13 150.3 mm to (245.5, 119.5)
- moved D2 147.9 mm to (248.5, 119.5), turned to 90 degrees
- moved LED2 146.4 mm to (235.8, 118.2), turned to 270 degrees
- moved P5 140.3 mm to (266.5, 120.0), turned to 270 degrees
- moved RV2 139.4 mm to (208.2, 108.2)
- moved RV1 138.5 mm to (208.2, 106.8)
- moved F1 138.5 mm to (211.6, 104.3)
- moved L1 135.5 mm to (208.2, 111.0), turned to 180 degrees
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Connections:
- C13 pad 1: VSS -> Net-(C13-Pad1)
- C3 pad 1: Net-(C3-Pad1) -> Net-(C13-Pad1)
- D2 pad 1: VSS -> Net-(C13-Pad1)
- P2 pad 2: VSS -> Net-(F2-Pad2)
- P7 pad 1: +5V -> SERVO
- P7 pad 2: SERVO -> +5V
- R1 pad 1: VSS -> +5V
- R1 pad 2: Net-(C3-Pad1) -> SCL
- R13 pad 1: +3V3 -> D-
- R13 pad 2: SCL -> Net-(P1-Pad2)
- R14 pad 1: +3V3 -> D+
- R14 pad 2: SDA -> Net-(P1-Pad3)
- R2 pad 1: Net-(C3-Pad1) -> +5V
- R2 pad 2: GND -> SDA
- U1 pad 1: Net-(Q1-Pad1) -> SDA
- U1 pad 2: +3V3 -> GND
- U1 pad 3: Net-(C3-Pad1) -> Net-(U1-Pad3)
- U1 pad 4: GND -> SCL
- U1 pad 5: (no net) -> +5V
- U1 pad 6: (no net) -> Net-(U1-Pad6)
- U1 pad 7: (no net) -> GND
- U1 pad 8: +5V -> GND
- U2 pad 1: Net-(U2-Pad1) -> Net-(P3-Pad1)
- U2 pad 12: ACCEL_INT -> Net-(U2-Pad12)
- U2 pad 25: BUTTON_A -> BUTTON_B
- U2 pad 26: BUTTON_B -> BUTTON_A
- U2 pad 38: Net-(P3-Pad4) -> Net-(P3-Pad5)
- U2 pad 39: Net-(P3-Pad3) -> Net-(P3-Pad4)
- U2 pad 40: Net-(P3-Pad2) -> Net-(P3-Pad3)
- U2 pad 41: Net-(P3-Pad1) -> Net-(P3-Pad2)
- U4 pad 1: (no net) -> Net-(C13-Pad1)
- U4 pad 2: (no net) -> GND
- U4 pad 3: (no net) -> +5V
- U5 pad 8: (no net) -> GND
- U7 pad 8: (no net) -> GND
Routing:
- net +5V: track 43.5 -> 278.4 mm, vias 0 -> 12
- net GND: track 11.5 -> 107.1 mm, vias 0 -> 20
- net BUTTON_A: track 0.00 -> 50.1 mm, vias 0 -> 2
- net VUSB: track 0.00 -> 47.4 mm, vias 0 -> 3
- net BUTTON_B: track 0.00 -> 42.5 mm, vias 0 -> 1
- net SDA: track 0.00 -> 39.8 mm, vias 0 -> 1
- net SCL: track 0.00 -> 38.7 mm, vias 0 -> 1
- net Net-(P6-Pad1): track 43.1 -> 16.0 mm
- net SERVO: track 0.00 -> 25.4 mm, vias 0 -> 1
- net Net-(P6-Pad2): track 37.1 -> 15.1 mm
- net Net-(C12-Pad1): track 0.00 -> 19.8 mm, vias 0 -> 2
- net Net-(R7-Pad2): track 0.00 -> 19.3 mm, vias 0 -> 2
- net JOYSTICK_X: track 0.00 -> 18.1 mm, vias 0 -> 1
- net RIN1: track 29.6 -> 47.3 mm, vias 0 -> 2
- net FIN1: track 27.8 -> 45.5 mm, vias 0 -> 2
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- added copper zone on B.Cu, net GND
Other:
- board outline added: 70 x 30 mm
- net class Default: trace_width 0.25 -> 0.2
- rule pad_to_mask_clearance: 0.2 -> 0
- board text added: "+"
- board text added: "-"
- board text added: "5V"
- board text added: "6-12 VDC"
- board text added: "A0"
- board text added: "A1"
- board text added: "A2"
- board text added: "A3"
- board text added: "A4"
- board text added: "A5"
- board text added: "D12"
- board text added: "D4"
- board text added: "D7"
- board text added: "DE '17"
- board text added: "GND"
- board text added: "ISP"
- board text added: "JX"
- board text added: "JY"
- board text added: "M0"
- board text added: "M1"
- board text added: "PCBs sponsored by OSHpark!!"
- board text added: "PWM5/13"
- board text added: "PWM6"
- board text added: "PWM9/10"
- board text added: "Patriot Companion"
- board text added: "RV1"
- board text added: "RV2"
- board text added: "RX"
- board text added: "SCL"
- board text added: "SDA"
- board text added: "SERVO"
- board text added: "SW1"
- board text added: "TEMP/HUM"
- board text added: "TX"
