File: Patriot_Companion/Patriot_Companion.sch (KiCad schematic (older format))
At the start: 82 parts, among them P1 USB_OTG, P2 POWER_IN, P3 I/O, P4 CONN_02X03, P5 MOTOR_1, P6 MOTOR_2, P7 SERVO_HEADER, Q1 FDN340P, SW1 SWITCH, SW2 SWITCH, SW3 SWITCH, U1 LM358, U2 ATMEGA32U4-A, U3 LP2985-33DBVR, U4 7805, U5 BD6212HFP-TR, U6 NXP_MMA8652FCR1, U7 BD6212HFP-TR, U8 Si7006, Y1 16M

Commit message: ISP done
Parts:
- removed 1u1, C23: C, Capacitors_SMD:C_0603_HandSoldering, symbol C
- removed C11: 1u, Capacitors_SMD:C_0603_HandSoldering, symbol C
- removed C17: 1u0, Capacitors_SMD:C_0603_HandSoldering, symbol C
- removed C18, C19, C22: 0u1, Capacitors_SMD:C_0603_HandSoldering, symbol C
- removed LED4, LED5, LED6, LED7, LED8: NeoPixel, DM_Custom:SR_CUSTOM_NEO_PIX, symbol NeoPixel
- removed P3: I/O, Pin_Headers:Pin_Header_Angled_1x04_Pitch1.27mm, symbol CONN_01X04
- removed Q1: FDN340P, TO_SOT_Packages_SMD:SOT-23_Handsoldering, symbol Q_PMOS_GDS
- removed R17, R18: R, Resistors_SMD:R_0603_HandSoldering, symbol R
- removed RV3: POT_Dual_Separate, DM_Custom:IM_joystick, symbol POT_Dual_Separate
- removed U1: LM358, DM_Custom:DM_CUSTOM_LM398_S08, symbol LM358
- removed U3: LP2985-33DBVR, DM_Custom:NB_Custom_S-L2985, symbol LT1761-3.3
- removed U4: 7805, DM_Custom:AZ_Custom_Mosfet, symbol 7805
- removed U6: NXP_MMA8652FCR1, DM_Custom:NXP_MMA8652FCR1_hand, symbol NXP_MMA8652FCR1
- removed U8: Si7006, DM_Custom:SM_Custom_Si7006, symbol Si7006
- added D5: LED, KiCad_Footprints:ZF_SMD_pol_0805, symbol LED
- added D6: D, KiCad_Footprints:ZF_SMD_pol_0805, symbol D
- added F2: Polyfuse, KiCad_Footprints:ZF_SMD_1812, symbol Polyfuse
- added P3: CONN_01X07, KiCad_Footprints:ZF_CONN_1x7-hdr, symbol CONN_01X07
- added R19: R, KiCad_Footprints:ZF_SMD_NonPol_0603, symbol R
- added U1: SHT30-DIS-B, KiCad_Footprints:ZF_IC_DFN8-050, symbol SHT30-DIS-B
- added U4: LF33CDT-TRY, KiCad_Footprints:ZF_SMD_DPAK, symbol LF33CDT-TRY
- added U9: joystick, KiCad_Footprints:ZF_JOYSTICK, symbol joystick
- C1, C12, C2, C20, C24, C4, C5, C7, C8, C9: footprint Capacitors_SMD:C_0603_HandSoldering -> KiCad_Footprints:ZF_SMD_NonPol_0603
- C10: footprint Capacitors_SMD:C_0603_HandSoldering -> KiCad_Footprints:ZF_SMD_NonPol_0603; RoHS (none) -> Yes; Subs Allowed (none) -> No
- C13, C14, C15, C16, C6: footprint SMD_Packages:SMD-1206_Pol -> KiCad_Footprints:ZF_SMD_pol_1206
- C21, C25: footprint Capacitors_SMD:C_0603_HandSoldering -> KiCad_Footprints:ZF_SMD_pol_1206; RoHS (none) -> Yes; Subs Allowed (none) -> No
- C3: value C -> 0u1; footprint Capacitors_SMD:C_0603_HandSoldering -> KiCad_Footprints:ZF_SMD_NonPol_0603; RoHS (none) -> Yes; Subs Allowed (none) -> No
- D1: footprint Diodes_SMD:D_1206 -> KiCad_Footprints:ZF_SMD_pol_1206
- D2: footprint Diodes_SMD:D_SOT-23_ANK -> KiCad_Footprints:ZF_SMD_pol_0805; RoHS (none) -> Yes; Subs Allowed (none) -> No
- D3, D4: footprint LEDs:LED_0805 -> KiCad_Footprints:ZF_SMD_pol_0805
- F1: footprint Resistors_SMD:R_1812_HandSoldering -> KiCad_Footprints:ZF_SMD_1812; RoHS (none) -> Yes; Subs Allowed (none) -> No
- L1, L2: footprint Resistors_SMD:R_0805_HandSoldering -> KiCad_Footprints:ZF_SMD_pol_0805
- P1: footprint Connectors:USB_Micro-B -> KiCad_Footprints:ZF_CONN_USB-MICRO-B-SMD-holes
- P2: footprint Connectors:BARREL_JACK -> KiCad_Footprints:ZF_CONN_POWER_1x2; RoHS (none) -> Yes; Subs Allowed (none) -> No
- P4: footprint Pin_Headers:Pin_Header_Angled_2x03_Pitch1.27mm -> KiCad_Footprints:ZF_CONN_3x2_noshroud; RoHS (none) -> Yes; Subs Allowed (none) -> No
- P5, P6: footprint Connectors_Terminal_Blocks:TerminalBlock_Pheonix_PT-3.5mm_2pol -> KiCad_Footprints:ZF_CONN_POWER_1x2; RoHS (none) -> Yes; Subs Allowed (none) -> No
- P7: footprint Pin_Headers:Pin_Header_Angled_1x03_Pitch1.27mm -> KiCad_Footprints:ZF_CONN_1x3_servo; RoHS (none) -> Yes; Subs Allowed (none) -> No
- R1, R2: value 10k -> R; footprint Resistors_SMD:R_0603_HandSoldering -> KiCad_Footprints:ZF_SMD_NonPol_0603; RoHS (none) -> Yes; Subs Allowed (none) -> No
- R10, R11, R12, R15, R16, R3, R4, R5, R6, R7, R8, R9, RV1, RV2: footprint Resistors_SMD:R_0603_HandSoldering -> KiCad_Footprints:ZF_SMD_NonPol_0603
- R13, R14: value 1k -> R; footprint Resistors_SMD:R_0603_HandSoldering -> KiCad_Footprints:ZF_SMD_NonPol_0603; RoHS (none) -> Yes; Subs Allowed (none) -> No
- SW1: footprint DM_Custom:DM_CUSTOM_B3FS-4 -> KiCad_Footprints:ZF_SW_LS38; RoHS (none) -> Yes; Subs Allowed (none) -> No
- SW2, SW3: footprint DM_Custom:DM_CUSTOM_B3FS-4 -> KiCad_Footprints:ZF_SW_Metal_Ball_Tactile; RoHS (none) -> Yes; Subs Allowed (none) -> No
- U2: footprint DM_Custom:LW_CUSTOM_ATMEGA32 -> KiCad_Footprints:ZF_IC_TQFP44-0-8; RoHS (none) -> Yes; Subs Allowed (none) -> No
Connections:
- net +5V: now also P7.2 (P2), R1.1, R2.1, D5.2 (A), D6.1 (K), U1.5 (VDD), U4.3 (Vout), U9.1 (L/R+), U9.8 (U/D+); no longer P7.1 (P1)
- net BUTTON_A: now also U2.26 ((T1/~OC4D~/ADC9)PD6); no longer U2.25 ((ICP2/ADC8)PD4)
- net BUTTON_B: now also U2.25 ((ICP2/ADC8)PD4); no longer U2.26 ((T1/~OC4D~/ADC9)PD6)
- net D+: now also R14.1
- net D-: now also R13.1
- net GND: now also R19.2, U1.2 (ADDR), U1.7 (R), U1.8 (GND), U4.2 (GND), U9.4 (GND), U9.5 (GND); no longer R2.2
- net JOYSTICK_X: now also U9.7 (L/R)
- net JOYSTICK_Y: now also U9.6 (U/D)
- net SCL: now also R1.2, P3.6 (P6), U1.4 (SCL); no longer R13.2
- net SDA: now also R2.2, P3.7 (P7), U1.1 (SDA); no longer R14.2
- net SERVO: now also P7.1 (P1); no longer P7.2 (P2)
- net VUSB: now also D6.2 (A)
- net at U2.1 ((INT6/AIN0)PE6): now also P3.1 (P1)
- net at U2.38 ((ADC5/TMS)PF5): now also P3.5 (P5)
- net at U2.39 ((ADC4/TCK)PF4): now also P3.4 (P4)
- net at U2.40 ((ADC1)PF1): now also P3.3 (P3)
- net at U2.41 ((ADC0)PF0): now also P3.2 (P2)
- net at P1.2 (D-), RV1.1: now also R13.2
- net at P1.3 (D+), RV2.1: now also R14.2
- removed net +3V3: R13.1, R14.1
- net ACCEL_INT: no longer names the net of U2.12 ((OC0A/OC1C/~RTS~/PCINT7)PB7)
- net VSS: no longer names the net of C13.1, D2.1 (K)
- net VSS: now also C3.1, F2.1, U4.1 (Vin); no longer P2.2 (P2), R1.1
- new net: F2.2, P2.2 (P2)
- new net: D5.1 (K), R19.1
Other:
- note added: "REGULATOR"
- note removed: "ACCELEROMETER"
- note removed: "EXTERNAL POWER SUPPLY"
- note removed: "I/O HEADER"
- note removed: "POWER SUPPLY AUTO SWITCHER"
- note removed: "TEMP/HUMIDITY SENSOR"
- moved on the sheet: C13, C15, C16, C20, C21, C24, C25, D2, P2, P5, P6, R11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

Commit message: added ISP programmer reset pull up
Parts:
- D3, D4, D5: symbol LED -> LED-RESCUE-Patriot_Companion
- P1: symbol USB_OTG -> USB_OTG-RESCUE-Patriot_Companion
Other:
- note added: "mysteriously not tied to 5V"
Changed lines of the file:
@@
 EESchema Schematic File Version 2
+LIBS:Patriot_Companion-rescue
 LIBS:power
 LIBS:device
@@
 LIBS:valves
 LIBS:Patriot_Companion-cache
-LIBS:DM_Custom
 EELAYER 25 0
 EELAYER END
@@
 $EndComp
 $Comp
-L USB_OTG P1
+L USB_OTG-RESCUE-Patriot_Companion P1
 U 1 1 58B7EAC7
 P 2100 9550
@@
 SDA
 $Comp
-L LED D4
+L LED-RESCUE-Patriot_Companion D4
 U 1 1 58B9EF6A
 P 7700 3900
@@
 $EndComp
 $Comp
-L LED D3
+L LED-RESCUE-Patriot_Companion D3
 U 1 1 58B9F11D
 P 7700 2200
@@
 $EndComp
 $Comp
-L LED D5
+L LED-RESCUE-Patriot_Companion D5
 U 1 1 5917919A
 P 19200 5300
@@
 Wire Wire Line
 	20450 1900 20900 1900
+Text Notes 1750 950  0    60   ~ 0
+mysteriously not tied to 5V
 $EndSCHEMATC
