File: Chua/Chua.kicad_pcb (KiCad board)
At the start: 2 copper layers, 0 parts

Commit message: chua pcb traces
Parts:
- added BT1: Battery_Cell, DM_Custom:DM_9V_ON_BOARD, B.Cu at (113.3, 77.5)
- added BT2: Battery_Cell, DM_Custom:DM_9V_ON_BOARD, B.Cu at (85.7, 77.5)
- added C1: C, Capacitors_SMD:C_0805_HandSoldering, F.Cu at (104.0, 106.0)
- added C2: C, Capacitors_SMD:C_0805_HandSoldering, F.Cu at (91.2, 115.0)
- added C3: C, Capacitors_SMD:C_0805_HandSoldering, F.Cu at (89.0, 99.0)
- added P1: CONN_01X03, Pin_Headers:Pin_Header_Straight_1x03_Pitch2.54mm, F.Cu at (124.0, 141.5)
- added R1: R, Resistors_SMD:R_0805_HandSoldering, F.Cu at (99.0, 118.3)
- added R2: R, Resistors_SMD:R_0805_HandSoldering, F.Cu at (110.0, 111.0)
- added R3: R, Resistors_SMD:R_0805_HandSoldering, F.Cu at (84.0, 109.3)
- added R4: R, Resistors_SMD:R_0805_HandSoldering, F.Cu at (100.0, 94.0)
- added R5: R, Resistors_SMD:R_0805_HandSoldering, F.Cu at (96.3, 89.0)
- added R6: R, Resistors_SMD:R_0805_HandSoldering, F.Cu at (92.3, 94.0)
- added R7: R, Resistors_SMD:R_0805_HandSoldering, F.Cu at (97.0, 106.0)
- added R8: R, Resistors_SMD:R_0805_HandSoldering, F.Cu at (108.0, 94.3)
- added R9: R, Resistors_SMD:R_0805_HandSoldering, F.Cu at (108.0, 100.0)
- added RV1: POT, DM_Custom:DM_POT_296, F.Cu at (110.0, 141.0)
- added RV2: POT, DM_Custom:DM_POT_296, F.Cu at (90.0, 140.0)
- added U1: TL082, DM_Custom:DM_TSSOP8, F.Cu at (98.0, 111.0)
- added U2: TL082, DM_Custom:DM_TSSOP8, F.Cu at (98.0, 100.0)
Routing:
- net /VCC-: track 0.00 -> 94.5 mm, vias 0 -> 2
- net /VCC+: track 0.00 -> 86.6 mm, vias 0 -> 2
- net Net-(C3-Pad1): track 0.00 -> 67.0 mm, vias 0 -> 2
- net Net-(C1-Pad2): track 0.00 -> 45.0 mm
- net Net-(C2-Pad1): track 0.00 -> 28.3 mm
- net Net-(R2-Pad2): track 0.00 -> 27.3 mm, vias 0 -> 2
- net Net-(R4-Pad1): track 0.00 -> 22.4 mm
- net Net-(C1-Pad1): track 0.00 -> 21.8 mm
- net Net-(R1-Pad2): track 0.00 -> 17.0 mm
- net Net-(R7-Pad1): track 0.00 -> 14.6 mm
- net Net-(R5-Pad1): track 0.00 -> 12.3 mm
- net Net-(R8-Pad1): track 0.00 -> 9.97 mm
- added copper zone on B.Cu, net GND
- added copper zone on F.Cu, net GND
Other:
- board outline added: 60 x 80 mm
