File: CodeKitty/CodeKittyNanoBreakout.kicad_pcb (KiCad board)
At the start: 2 copper layers, 17.8 x 43.2 mm, 14 parts, among them P1 CONN_01X02, P2 CONN_01X02, P3 CONN_01X03, P4 CONN_01X03, P5 CONN_01X02, SW1 SW_PUSH_SMALL_H, SW2 Switch_SPDT_x2, U1 ArduinoNano

Commit message: updated CK board
Parts:
- moved SW1 0.22 mm to (203.9, 84.5), turned to 0 degrees
Routing:
- net GND: track 26.9 -> 22.0 mm
- net RST: track 40.5 -> 44.5 mm
- net Net-(P2-Pad2): track 8.13 -> 8.66 mm
Changed lines of the file:
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@@
   (general
     (links 25)
-    (no_connects 25)
+    (no_connects 0)
     (area 196.774999 82.474999 214.705001 125.805001)
     (thickness 1.6)
     (drawings 21)
-    (tracks 82)
+    (tracks 86)
     (zones 0)
     (modules 14)
@@
     (38 B.Mask user)
     (39 F.Mask user)
-    (40 Dwgs.User user hide)
-    (41 Cmts.User user hide)
-    (42 Eco1.User user hide)
-    (43 Eco2.User user hide)
+    (40 Dwgs.User user)
+    (41 Cmts.User user)
+    (42 Eco1.User user)
+    (43 Eco2.User user)
     (44 Edge.Cuts user)
-    (45 Margin user hide)
-    (46 B.CrtYd user hide)
-    (47 F.CrtYd user hide)
-    (48 B.Fab user hide)
-    (49 F.Fab user hide)
+    (45 Margin user)
+    (46 B.CrtYd user)
+    (47 F.CrtYd user)
+    (48 B.Fab user)
+    (49 F.Fab user)
   )
   (setup
@@
       (net 3 GND))
   )
-  (module DM_Custom:DM_SMD_BUTTON_PTS810 (layer F.Cu)
-    (at 203.7 84.35 180)
-    (fp_text reference SW1 (at -0.05 7.7 180) (layer F.SilkS)
-      (effects (font (size 1 1) (thickness 0.15)))
-    )
-    (fp_text value SW_PUSH_SMALL_H (at 0 -7.55 180) (layer F.Fab)
-      (effects (font (size 1 1) (thickness 0.15)))
-    )
-    (fp_line (start -2.1 1.6) (end 2.1 1.6) (layer F.SilkS) (width 0.15))
-    (fp_line (start -2.1 -1.6) (end -2.1 1.6) (layer F.SilkS) (width 0.15))
-    (fp_line (start 2.1 -1.6) (end -2.1 -1.6) (layer F.SilkS) (width 0.15))
-    (fp_line (start 2.1 1.6) (end 2.1 -1.6) (layer F.SilkS) (width 0.15))
-    (pad 1 thru_hole rect (at -2.45 -1 180) (size 1.8 1) (drill 0.762) (layers *.Cu *.Mask)
-      (net 33 RST))
-    (pad 1 thru_hole rect (at 2.45 -1 180) (size 1.8 1) (drill 0.762) (layers *.Cu *.Mask)
-      (net 33 RST))
-    (pad 2 thru_hole rect (at 2.45 1 180) (size 1.8 1) (drill 0.762) (layers *.Cu *.Mask)
-      (net 3 GND))
-    (pad 2 thru_hole rect (at -2.45 1 180) (size 1.8 1) (drill 0.762) (layers *.Cu *.Mask)
-      (net 3 GND))
-  )
   (module DM_Custom:DM_SPDT_RTAngle_JS102011SAQN (layer B.Cu)
     (at 203.8 84.45)
@@
     (pad "" np_thru_hole circle (at 3.4 0) (size 0.9 0.9) (drill 0.9) (layers *.Cu *.Mask))
   )
+  (module DM_Custom:DM_SMD_BUTTON_PTS810 (layer F.Cu)
+    (at 203.9 84.45)
+    (fp_text reference SW1 (at -0.1 -0.1) (layer F.SilkS)
+      (effects (font (size 1 1) (thickness 0.15)))
+    )
+    (fp_text value SW_PUSH_SMALL_H (at 0 -7.55) (layer F.Fab)
+      (effects (font (size 1 1) (thickness 0.15)))
+    )
+    (fp_line (start -2.1 1.6) (end 2.1 1.6) (layer F.SilkS) (width 0.15))
+    (fp_line (start -2.1 -1.6) (end -2.1 1.6) (layer F.SilkS) (width 0.15))
+    (fp_line (start 2.1 -1.6) (end -2.1 -1.6) (layer F.SilkS) (width 0.15))
+    (fp_line (start 2.1 1.6) (end 2.1 -1.6) (layer F.SilkS) (width 0.15))
+    (pad 1 smd rect (at -2.45 -1) (size 1.8 1) (layers F.Cu F.Paste F.Mask)
+      (net 33 RST))
+    (pad 1 smd rect (at 2.45 -1) (size 1.8 1) (layers F.Cu F.Paste F.Mask)
+      (net 33 RST))
+    (pad 2 smd rect (at 2.45 1) (size 1.8 1) (layers F.Cu F.Paste F.Mask)
+      (net 3 GND))
+    (pad 2 smd rect (at -2.45 1) (size 1.8 1) (layers F.Cu F.Paste F.Mask)
+      (net 3 GND))
+  )
   (gr_text S (at 201.6 100.55) (layer F.SilkS)
     (effects (font (size 1.5 1.5) (thickness 0.3)))
@@
   (segment (start 211.6 85.55) (end 211.6 83.65) (width 0.3048) (layer F.Cu) (net 1))
   (segment (start 209.5 86) (end 211.15 86) (width 0.3048) (layer F.Cu) (net 1))
-  (segment (start 208.9 83.65) (end 208.9 84.25) (width 0.3048) (layer F.Cu) (net 2))
-  (segment (start 208.9 84.25) (end 207.7 85.45) (width 0.3048) (layer F.Cu) (net 2))
-  (via (at 207.7 85.45) (size 0.6858) (drill 0.3302) (layers F.Cu B.Cu) (net 2))
+  (segment (start 208.9 83.65) (end 208.9 84.65) (width 0.3048) (layer F.Cu) (net 2))
+  (segment (start 208.9 84.65) (end 208.1 85.45) (width 0.3048) (layer F.Cu) (net 2))
+  (segment (start 209.5 103.15) (end 208.1 101.75) (width 0.3048) (layer B.Cu) (net 2))
+  (segment (start 208.1 101.75) (end 208.1 101.45) (width 0.3048) (layer B.Cu) (net 2))
+  (via (at 208.1 85.45) (size 0.6858) (drill 0.3302) (layers F.Cu B.Cu) (net 2))
   (segment (start 205.7 103.15) (end 209.5 103.15) (width 0.508) (layer B.Cu) (net 2))
   (segment (start 211.7 105.35) (end 209.5 103.15) (width 0.508) (layer B.Cu) (net 2))
   (segment (start 211.7 112.63) (end 211.7 105.35) (width 0.508) (layer B.Cu) (net 2))
   (segment (start 213.32 114.25) (end 211.7 112.63) (width 0.508) (layer B.Cu) (net 2))
-  (segment (start 207.7 85.45) (end 207.7 101.35) (width 0.3048) (layer B.Cu) (net 2))
-  (segment (start 207.7 101.35) (end 209.5 103.15) (width 0.3048) (layer B.Cu) (net 2))
+  (segment (start 208.1 85.55) (end 208.1 101.45) (width 0.3048) (layer B.Cu) (net 2))
   (segment (start 206.3 98.25) (end 205.6 97.55) (width 0.3048) (layer F.Cu) (net 3))
   (segment (start 205.6 97.55) (end 205.6 94.45) (width 0.3048) (layer F.Cu) (net 3))
@@
   (segment (start 201.1 114.35) (end 201.1 111.45) (width 0.3048) (layer B.Cu) (net 3))
   (via (at 201.1 111.45) (size 0.6858) (drill 0.3302) (layers F.Cu B.Cu) (net 3))
-  (segment (start 201.25 83.35) (end 206.15 83.35) (width 0.3048) (layer F.Cu) (net 3))
   (segment (start 200.4 108.85) (end 213.32 121.77) (width 0.508) (layer B.Cu) (net 4))
   (segment (start 213.32 121.77) (end 213.32 121.87) (width 0.508) (layer B.Cu) (net 4))
@@
   (segment (start 201.5 96.25) (end 201.5 97.648) (width 0.508) (layer B.Cu) (net 4))
   (segment (start 201.5 97.648) (end 199.6 99.548) (width 0.508) (layer B.Cu) (net 4))
-  (segment (start 208.3477 87.35) (end 208.3477 87.5477) (width 0.3048) (layer B.Cu) (net 5))
-  (segment (start 208.3477 87.5477) (end 209.5 88.7) (width 0.3048) (layer B.Cu) (net 5))
-  (segment (start 206.9 89.15) (end 206.9 88.7977) (width 0.3048) (layer F.Cu) (net 5))
-  (segment (start 206.9 88.7977) (end 208.3477 87.35) (width 0.3048) (layer F.Cu) (net 5))
-  (via (at 208.3477 87.35) (size 0.6858) (drill 0.3302) (layers F.Cu B.Cu) (net 5))
-  (segment (start 206.96 90.55) (end 206.96 89.21) (width 0.3048) (layer B.Cu) (net 5))
-  (segment (start 206.96 89.21) (end 206.9 89.15) (width 0.3048) (layer B.Cu) (net 5))
-  (via (at 206.9 89.15) (size 0.6858) (drill 0.3302) (layers F.Cu B.Cu) (net 5))
+  (segment (start 209.5 87.35) (end 208.760001 87.35) (width 0.3048) (layer F.Cu) (net 5))
+  (segment (start 208.760001 87.35) (end 206.96 89.150001) (width 0.3048) (layer F.Cu) (net 5))
+  (via (at 206.96 89.150001) (size 0.6858) (drill 0.3302) (layers F.Cu B.Cu) (net 5))
+  (segment (start 209.05 88.7) (end 209.5 88.25) (width 0.3048) (layer B.Cu) (net 5))
+  (segment (start 209.5 88.25) (end 209.5 87.35) (width 0.3048) (layer B.Cu) (net 5))
+  (via (at 209.5 87.35) (size 0.6858) (drill 0.3302) (layers F.Cu B.Cu) (net 5))
+  (segment (start 209.5 88.7) (end 209.05 88.7) (width 0.3048) (layer B.Cu) (net 5))
+  (segment (start 206.96 90.55) (end 206.96 89.150001) (width 0.3048) (layer B.Cu) (net 5))
+  (segment (start 206.96 89.21) (end 206.96 89.150001) (width 0.3048) (layer B.Cu) (net 5))
   (segment (start 205.6 91.91) (end 206.96 90.55) (width 0.3048) (layer B.Cu) (net 5))
-  (segment (start 209.5 88.7) (end 210.05 88.7) (width 0.3048) (layer B.Cu) (net 5))
   (segment (start 205.7 100.61) (end 199.02 93.93) (width 0.3048) (layer F.Cu) (net 6))
   (segment (start 199.02 93.93) (end 198.08 93.93) (width 0.3048) (layer F.Cu) (net 6))
@@
   (segment (start 203.8 88.55) (end 204.5 89.25) (width 0.3048) (layer B.Cu) (net 32))
   (via (at 204.5 89.25) (size 0.6858) (drill 0.3302) (layers F.Cu B.Cu) (net 32))
+  (segment (start 201.45 83.45) (end 202.6548 83.45) (width 0.3048) (layer F.Cu) (net 33))
+  (segment (start 202.6548 83.45) (end 206.35 83.45) (width 0.3048) (layer F.Cu) (net 33))
+  (segment (start 201.45 83.45) (end 200.2452 83.45) (width 0.3048) (layer F.Cu) (net 33))
+  (segment (start 200.2452 83.45) (end 199.645199 84.050001) (width 0.3048) (layer F.Cu) (net 33))
+  (segment (start 199.645199 84.050001) (end 199.645199 91.595199) (width 0.3048) (layer F.Cu) (net 33))
+  (segment (start 199.645199 91.595199) (end 201.25 93.2) (width 0.3048) (layer F.Cu) (net 33))
   (segment (start 199.7 111.75) (end 199.7 115.17) (width 0.3048) (layer F.Cu) (net 33))
   (segment (start 199.7 115.17) (end 198.08 116.79) (width 0.3048) (layer F.Cu) (net 33))
@@
   (segment (start 199.7 101.65) (end 199.7 111.75) (width 0.3048) (layer B.Cu) (net 33))
   (via (at 199.7 111.75) (size 0.6858) (drill 0.3302) (layers F.Cu B.Cu) (net 33))
-  (segment (start 201.25 85.35) (end 201.25 93.2) (width 0.3048) (layer F.Cu) (net 33))
   (segment (start 201.25 93.2) (end 204.7 96.65) (width 0.3048) (layer F.Cu) (net 33))
   (via (at 204.7 96.65) (size 0.6858) (drill 0.3302) (layers F.Cu B.Cu) (net 33))
-  (segment (start 201.25 85.35) (end 206.15 85.35) (width 0.3048) (layer F.Cu) (net 33))
   (zone (net 3) (net_name GND) (layer F.Cu) (hatch edge 0.508)
     (connect_pads (clearance 0.508))

Commit message: kitty3
Parts:
- P5: value CONN_01X02 -> CONN_01X03; footprint Pin_Headers:Pin_Header_Straight_1x02_Pitch2.54mm -> Pin_Headers:Pin_Header_Straight_1x03_Pitch2.54mm; moved to F.Cu
- moved P5 0.16 mm to (201.6, 105.5), turned to 180 degrees
Connections:
- P5 pad 2: BUZZ -> 5V
- U1 pad 20: Net-(U1-Pad20) -> SENS
Routing:
- net RST: track 44.5 -> 22.5 mm, vias 2 -> 1
- net BUZZ: track 32.1 -> 29.2 mm
