File: CodeKitty/CodeKittyNanoBreakout.sch (KiCad schematic (older format))
At the start: 10 parts, among them P1 CONN_01X02, P2 CONN_01X02, P3 CONN_01X03, P4 CONN_01X03, P5 CONN_01X02, U1 ArduinoNano

Commit message: update of codekitty
Parts:
- removed R3: R, Resistors_SMD:R_0805_HandSoldering, symbol R
- added F1: F_Small, DM_Custom:DM_FUSE_PTC0ZCG, symbol F_Small
- added SP1: SPEAKER, DM_Custom:DM_PiezSMD_PMKCS0909E4000-R1, symbol SPEAKER
- added SW1: SW_PUSH_SMALL_H, DM_Custom:DM_SMD_BUTTON_PTS810, symbol SW_PUSH_SMALL_H
- added SW2: Switch_SPDT_x2, DM_Custom:DM_SPDT_RTAngle_JS102011SAQN, symbol Switch_SPDT_x2
Connections:
- net BUZZ: now also P5.2 (P2), SP1.1
- net GND: now also SP1.2, SW1.2
- net VCC: now also F1.2; no longer P1.2 (P2)
- net RST: now reaches U1.3 (RESET)
- net RST: now also SW1.1
- new net: P1.2 (P2), SW2.2 (B)
- new net: F1.1, SW2.3 (C)
Other:
- moved on the sheet: D1, P1, R1
Changed lines of the file:
@@
 LIBS:valves
 LIBS:DM_Custom
+LIBS:CodeKittyNanoBreakout-cache
 EELAYER 25 0
 EELAYER END
@@
 L CONN_01X02 P1
 U 1 1 597FBC27
-P 1625 1900
-F 0 "P1" H 1625 2050 50  0000 C CNN
-F 1 "CONN_01X02" V 1725 1900 50  0000 C CNN
-F 2 "Pin_Headers:Pin_Header_Straight_1x02_Pitch2.54mm" H 1625 1900 50  0001 C CNN
-F 3 "" H 1625 1900 50  0000 C CNN
-	1    1625 1900
+P 1625 1375
+F 0 "P1" H 1625 1525 50  0000 C CNN
+F 1 "CONN_01X02" V 1725 1375 50  0000 C CNN
+F 2 "Pin_Headers:Pin_Header_Straight_1x02_Pitch2.54mm" H 1625 1375 50  0001 C CNN
+F 3 "" H 1625 1375 50  0000 C CNN
+	1    1625 1375
 	0    -1   -1   0
 $EndComp
@@
 Text GLabel 6225 4125 0    39   Input ~ 0
 RSERVO
-Text Notes 1125 1525 0    197  ~ 0
+Text Notes 1175 1050 0    197  ~ 0
 POWER
-Text GLabel 1675 2100 3    39   Input ~ 0
+Text GLabel 2550 1675 2    39   Input ~ 0
 VCC
-Text GLabel 1575 2100 3    39   Input ~ 0
-GND
 $Comp
 L CONN_01X02 P5
@@
 L LED D1
 U 1 1 597FE136
-P 1650 2600
-F 0 "D1" H 1650 2700 50  0000 C CNN
-F 1 "LED" H 1650 2500 50  0000 C CNN
-F 2 "LEDs:LED_0805_HandSoldering" H 1650 2600 50  0001 C CNN
-F 3 "" H 1650 2600 50  0000 C CNN
-	1    1650 2600
+P 1650 3525
+F 0 "D1" H 1650 3625 50  0000 C CNN
+F 1 "LED" H 1650 3425 50  0000 C CNN
+F 2 "LEDs:LED_0805_HandSoldering" H 1650 3525 50  0001 C CNN
+F 3 "" H 1650 3525 50  0000 C CNN
+	1    1650 3525
 	-1   0    0    1
 $EndComp
@@
 L R R1
 U 1 1 597FE2C9
-P 1950 2875
-F 0 "R1" V 2030 2875 50  0000 C CNN
-F 1 "R" V 1950 2875 50  0000 C CNN
-F 2 "Resistors_SMD:R_0805_HandSoldering" V 1880 2875 50  0001 C CNN
-F 3 "" H 1950 2875 50  0000 C CNN
-	1    1950 2875
-	1    0    0    -1
-$EndComp
-Text GLabel 1450 2600 0    39   Input ~ 0
-5V
-Text GLabel 1950 3025 3    39   Input ~ 0
-GND
-Wire Wire Line
-	1950 2725 1950 2600
-Wire Wire Line
-	1950 2600 1850 2600
-$Comp
-L R R3
-U 1 1 597FE6DF
-P 8700 1675
-F 0 "R3" V 8780 1675 50  0000 C CNN
-F 1 "R" V 8700 1675 50  0000 C CNN
-F 2 "Resistors_SMD:R_0805_HandSoldering" V 8630 1675 50  0001 C CNN
-F 3 "" H 8700 1675 50  0000 C CNN
-	1    8700 1675
-	0    1    1    0
-$EndComp
-Wire Wire Line
-	8550 1675 8525 1675
+P 1950 3800
+F 0 "R1" V 2030 3800 50  0000 C CNN
+F 1 "R" V 1950 3800 50  0000 C CNN
+F 2 "Resistors_SMD:R_0805_HandSoldering" V 1880 3800 50  0001 C CNN
+F 3 "" H 1950 3800 50  0000 C CNN
+	1    1950 3800
+	1    0    0    -1
+$EndComp
+Text GLabel 1450 3525 0    39   Input ~ 0
+5V
+Text GLabel 1950 3950 3    39   Input ~ 0
+GND
+Wire Wire Line
+	1950 3650 1950 3525
+Wire Wire Line
+	1950 3525 1850 3525
+Wire Wire Line
+	8525 1675 8900 1675
 Wire Wire Line
 	8525 1675 8525 1550
-Wire Wire Line
-	8900 1675 8850 1675
+Text GLabel 1575 1575 3    39   Input ~ 0
+GND
+$Comp
+L F_Small F1
+U 1 1 59DC1D02
+P 2375 1675
+F 0 "F1" H 2335 1735 50  0000 L CNN
+F 1 "F_Small" H 2255 1615 50  0000 L CNN
+F 2 "DM_Custom:DM_FUSE_PTC0ZCG" H 2375 1675 50  0001 C CNN
+F 3 "" H 2375 1675 50  0000 C CNN
+	1    2375 1675
+	1    0    0    -1
+$EndComp
+Wire Wire Line
+	2475 1675 2550 1675
+$Comp
+L Switch_SPDT_x2 SW2
+U 1 1 59DC2380
+P 1975 1575
+F 0 "SW2" H 1775 1725 50  0000 C CNN
+F 1 "Switch_SPDT_x2" H 1725 1425 50  0000 C CNN
+F 2 "DM_Custom:DM_SPDT_RTAngle_JS102011SAQN" H 1975 1575 50  0001 C CNN
+F 3 "" H 1975 1575 50  0000 C CNN
+	1    1975 1575
+	1    0    0    -1
+$EndComp
+$Comp
+L SPEAKER SP1
+U 1 1 59DC25FB
+P 8925 2350
+F 0 "SP1" H 8825 2600 50  0000 C CNN
+F 1 "SPEAKER" H 8825 2100 50  0000 C CNN
+F 2 "DM_Custom:DM_PiezSMD_PMKCS0909E4000-R1" H 8925 2350 50  0001 C CNN
+F 3 "" H 8925 2350 50  0000 C CNN
+	1    8925 2350
+	1    0    0    -1
+$EndComp
+Text GLabel 8625 2250 0    39   Input ~ 0
+BUZZ
+Text GLabel 8625 2450 0    39   Input ~ 0
+GND
+$Comp
+L SW_PUSH_SMALL_H SW1
+U 1 1 59DC272F
+P 1675 2475
+F 0 "SW1" H 1755 2585 50  0000 C CNN
+F 1 "SW_PUSH_SMALL_H" H 2035 2415 50  0000 C CNN
+F 2 "DM_Custom:DM_SMD_BUTTON_PTS810" H 1675 2675 50  0001 C CNN
+F 3 "" H 1675 2675 50  0000 C CNN
+	1    1675 2475
+	1    0    0    -1
+$EndComp
+Text GLabel 3150 2300 0    39   Input ~ 0
+RST
+Text GLabel 1525 2475 0    39   Input ~ 0
+RST
+Text GLabel 1825 2475 2    39   Input ~ 0
+GND
 $EndSCHEMATC

Commit message: kitty3
Parts:
- removed P5: CONN_01X02, Pin_Headers:Pin_Header_Straight_1x02_Pitch2.54mm, symbol CONN_01X02
- added P5: CONN_01X03, Pin_Headers:Pin_Header_Straight_1x03_Pitch2.54mm, symbol CONN_01X03
Connections:
- net 5V: now also P5.2 (P2)
- net GND: now also P5.1 (P1)
- net SENS: now reaches U1.20 (A1)
- net SENS: now also P5.3 (P3)
Other:
- moved on the sheet: SP1
Changed lines of the file:
@@
 Text GLabel 2550 1675 2    39   Input ~ 0
 VCC
-$Comp
-L CONN_01X02 P5
-U 1 1 597FDB7A
-P 8475 1350
-F 0 "P5" H 8475 1500 50  0000 C CNN
-F 1 "CONN_01X02" V 8575 1350 50  0000 C CNN
-F 2 "Pin_Headers:Pin_Header_Straight_1x02_Pitch2.54mm" H 8475 1350 50  0001 C CNN
-F 3 "" H 8475 1350 50  0000 C CNN
-	1    8475 1350
-	0    -1   -1   0
-$EndComp
-Text GLabel 8425 1550 3    39   Input ~ 0
+Text GLabel 8750 3175 0    39   Input ~ 0
 GND
-Text GLabel 8900 1675 2    39   Input ~ 0
-BUZZ
-Text Notes 7875 1125 0    197  ~ 0
+Text Notes 7900 1125 0    197  ~ 0
 SPEAKER
 $Comp
@@
 Wire Wire Line
 	1950 3525 1850 3525
-Wire Wire Line
-	8525 1675 8900 1675
-Wire Wire Line
-	8525 1675 8525 1550
 Text GLabel 1575 1575 3    39   Input ~ 0
 GND
@@
 L SPEAKER SP1
 U 1 1 59DC25FB
-P 8925 2350
-F 0 "SP1" H 8825 2600 50  0000 C CNN
-F 1 "SPEAKER" H 8825 2100 50  0000 C CNN
-F 2 "DM_Custom:DM_PiezSMD_PMKCS0909E4000-R1" H 8925 2350 50  0001 C CNN
-F 3 "" H 8925 2350 50  0000 C CNN
-	1    8925 2350
+P 8775 1850
+F 0 "SP1" H 8675 2100 50  0000 C CNN
+F 1 "SPEAKER" H 8675 1600 50  0000 C CNN
+F 2 "DM_Custom:DM_PiezSMD_PMKCS0909E4000-R1" H 8775 1850 50  0001 C CNN
+F 3 "" H 8775 1850 50  0000 C CNN
+	1    8775 1850
 	1    0    0    -1
 $EndComp
-Text GLabel 8625 2250 0    39   Input ~ 0
+Text GLabel 8475 1750 0    39   Input ~ 0
 BUZZ
-Text GLabel 8625 2450 0    39   Input ~ 0
+Text GLabel 8475 1950 0    39   Input ~ 0
 GND
 $Comp
@@
 Text GLabel 1825 2475 2    39   Input ~ 0
 GND
+$Comp
+L CONN_01X03 P5
+U 1 1 59FFB57F
+P 8950 3275
+F 0 "P5" H 8950 3475 50  0000 C CNN
+F 1 "CONN_01X03" V 9050 3275 50  0000 C CNN
+F 2 "Pin_Headers:Pin_Header_Straight_1x03_Pitch2.54mm" H 8950 3275 50  0001 C CNN
+F 3 "" H 8950 3275 50  0000 C CNN
+	1    8950 3275
+	1    0    0    -1
+$EndComp
+Text GLabel 8750 3275 0    39   Input ~ 0
+5V
+Text GLabel 8750 3375 0    39   Input ~ 0
+SENS
+Text GLabel 4750 3100 2    39   Input ~ 0
+SENS
 $EndSCHEMATC
