File: CodeKitty/CodeKittyNanoBreakout.sch (KiCad schematic (older format))
At the start: 13 parts, among them P1 CONN_01X02, P2 CONN_01X02, P3 CONN_01X03, P4 CONN_01X03, P5 CONN_01X03, SW1 SW_PUSH_SMALL_H, SW2 Switch_SPDT_x2, U1 ArduinoNano

Commit message: some cknano
Other:
- note added: "SENSORS"
Changed lines of the file:
@@
 Text GLabel 4750 3100 2    39   Input ~ 0
 SENS
+Text Notes 7925 2950 0    197  ~ 0
+SENSORS
 $EndSCHEMATC

Commit message: getting to 1.0
Parts:
- added D?: D, symbol D
- added Q?: MMBT3904, SOT-23, symbol MMBT3904
- added R? (x2): R, symbol R
Connections:
- net 5V: now also SP1.1, R?.1
- net BUZZ: now also R?.2; no longer SP1.1
- net GND: now also Q?.2 (E); no longer SP1.2
- new net: D?.2 (A), Q?.3 (C), SP1.2
- new net: D?.1 (K), R?.2
- new net: Q?.1 (B), R?.1
Other:
- moved on the sheet: SP1
Changed lines of the file:
@@
 Text GLabel 8750 3175 0    39   Input ~ 0
 GND
-Text Notes 7900 1125 0    197  ~ 0
+Text Notes 8225 875  0    197  ~ 0
 SPEAKER
 $Comp
@@
 L SPEAKER SP1
 U 1 1 59DC25FB
-P 8775 1850
-F 0 "SP1" H 8675 2100 50  0000 C CNN
-F 1 "SPEAKER" H 8675 1600 50  0000 C CNN
-F 2 "DM_Custom:DM_PiezSMD_PMKCS0909E4000-R1" H 8775 1850 50  0001 C CNN
-F 3 "" H 8775 1850 50  0000 C CNN
-	1    8775 1850
+P 9975 1550
+F 0 "SP1" H 9875 1800 50  0000 C CNN
+F 1 "SPEAKER" H 9875 1300 50  0000 C CNN
+F 2 "DM_Custom:DM_PiezSMD_PMKCS0909E4000-R1" H 9975 1550 50  0001 C CNN
+F 3 "" H 9975 1550 50  0000 C CNN
+	1    9975 1550
 	1    0    0    -1
 $EndComp
-Text GLabel 8475 1750 0    39   Input ~ 0
+Text GLabel 8450 2100 0    39   Input ~ 0
 BUZZ
-Text GLabel 8475 1950 0    39   Input ~ 0
+Text GLabel 8450 2450 0    39   Input ~ 0
 GND
 $Comp
@@
 Text Notes 7925 2950 0    197  ~ 0
 SENSORS
+Text GLabel 8425 1300 0    39   Input ~ 0
+5V
+$Comp
+L D D?
+U 1 1 5A0CCEA3
+P 9150 1650
+F 0 "D?" H 9150 1750 50  0000 C CNN
+F 1 "D" H 9150 1550 50  0000 C CNN
+F 2 "" H 9150 1650 50  0000 C CNN
+F 3 "" H 9150 1650 50  0000 C CNN
+	1    9150 1650
+	1    0    0    -1
+$EndComp
+$Comp
+L R R?
+U 1 1 5A0CCF8E
+P 8675 1475
+F 0 "R?" V 8755 1475 50  0000 C CNN
+F 1 "R" V 8675 1475 50  0000 C CNN
+F 2 "" V 8605 1475 50  0000 C CNN
+F 3 "" H 8675 1475 50  0000 C CNN
+	1    8675 1475
+	1    0    0    -1
+$EndComp
+$Comp
+L R R?
+U 1 1 5A0CD00D
+P 8875 2100
+F 0 "R?" V 8955 2100 50  0000 C CNN
+F 1 "R" V 8875 2100 50  0000 C CNN
+F 2 "" V 8805 2100 50  0000 C CNN
+F 3 "" H 8875 2100 50  0000 C CNN
+	1    8875 2100
+	0    1    1    0
+$EndComp
+$Comp
+L MMBT3904 Q?
+U 1 1 5A0CD092
+P 9325 2100
+F 0 "Q?" H 9525 2175 50  0000 L CNN
+F 1 "MMBT3904" H 9525 2100 50  0000 L CNN
+F 2 "SOT-23" H 9525 2025 50  0000 L CIN
+F 3 "" H 9325 2100 50  0000 L CNN
+	1    9325 2100
+	1    0    0    -1
+$EndComp
+Wire Wire Line
+	8450 2450 9425 2450
+Wire Wire Line
+	9425 2450 9425 2300
+Wire Wire Line
+	9025 2100 9125 2100
+Wire Wire Line
+	8450 2100 8725 2100
+Wire Wire Line
+	9675 1650 9300 1650
+Wire Wire Line
+	9425 1900 9425 1650
+Connection ~ 9425 1650
+Wire Wire Line
+	9000 1650 8675 1650
+Wire Wire Line
+	8675 1650 8675 1625
+Wire Wire Line
+	8675 1325 9675 1325
+Wire Wire Line
+	9675 1325 9675 1450
+Wire Wire Line
+	8425 1300 9275 1300
+Wire Wire Line
+	9275 1300 9275 1325
+Connection ~ 9275 1325
 $EndSCHEMATC

Commit message: ServoTester first commit
Parts:
- D2: renamed from D?; footprint (none) -> Diodes_SMD:D_SOD-323_HandSoldering
- Q1: renamed from Q?; footprint SOT-23 -> TO_SOT_Packages_SMD:SOT-23
- R1, R2: footprint Resistors_SMD:R_0805_HandSoldering -> Resistors_SMD:R_0603_HandSoldering
- R3, R4: renamed from R?; footprint (none) -> Resistors_SMD:R_0603_HandSoldering
Changed lines of the file:
@@
 F 0 "R2" V 6755 1650 50  0000 C CNN
 F 1 "R" V 6675 1650 50  0000 C CNN
-F 2 "Resistors_SMD:R_0805_HandSoldering" V 6605 1650 50  0001 C CNN
+F 2 "Resistors_SMD:R_0603_HandSoldering" V 6605 1650 50  0001 C CNN
 F 3 "" H 6675 1650 50  0000 C CNN
 	1    6675 1650
@@
 F 0 "R1" V 2030 3800 50  0000 C CNN
 F 1 "R" V 1950 3800 50  0000 C CNN
-F 2 "Resistors_SMD:R_0805_HandSoldering" V 1880 3800 50  0001 C CNN
+F 2 "Resistors_SMD:R_0603_HandSoldering" V 1880 3800 50  0001 C CNN
 F 3 "" H 1950 3800 50  0000 C CNN
 	1    1950 3800
@@
 5V
 $Comp
-L D D?
+L D D2
 U 1 1 5A0CCEA3
 P 9150 1650
-F 0 "D?" H 9150 1750 50  0000 C CNN
+F 0 "D2" H 9150 1750 50  0000 C CNN
 F 1 "D" H 9150 1550 50  0000 C CNN
-F 2 "" H 9150 1650 50  0000 C CNN
+F 2 "Diodes_SMD:D_SOD-323_HandSoldering" H 9150 1650 50  0001 C CNN
 F 3 "" H 9150 1650 50  0000 C CNN
 	1    9150 1650
@@
 $EndComp
 $Comp
-L R R?
+L R R3
 U 1 1 5A0CCF8E
 P 8675 1475
-F 0 "R?" V 8755 1475 50  0000 C CNN
+F 0 "R3" V 8755 1475 50  0000 C CNN
 F 1 "R" V 8675 1475 50  0000 C CNN
-F 2 "" V 8605 1475 50  0000 C CNN
+F 2 "Resistors_SMD:R_0603_HandSoldering" V 8605 1475 50  0001 C CNN
 F 3 "" H 8675 1475 50  0000 C CNN
 	1    8675 1475
@@
 $EndComp
 $Comp
-L R R?
+L R R4
 U 1 1 5A0CD00D
 P 8875 2100
-F 0 "R?" V 8955 2100 50  0000 C CNN
+F 0 "R4" V 8955 2100 50  0000 C CNN
 F 1 "R" V 8875 2100 50  0000 C CNN
-F 2 "" V 8805 2100 50  0000 C CNN
+F 2 "Resistors_SMD:R_0603_HandSoldering" V 8805 2100 50  0001 C CNN
 F 3 "" H 8875 2100 50  0000 C CNN
 	1    8875 2100
@@
 $EndComp
 $Comp
-L MMBT3904 Q?
+L MMBT3904 Q1
 U 1 1 5A0CD092
 P 9325 2100
-F 0 "Q?" H 9525 2175 50  0000 L CNN
+F 0 "Q1" H 9525 2175 50  0000 L CNN
 F 1 "MMBT3904" H 9525 2100 50  0000 L CNN
-F 2 "SOT-23" H 9525 2025 50  0000 L CIN
+F 2 "TO_SOT_Packages_SMD:SOT-23" H 9525 2025 50  0000 L CIN
 F 3 "" H 9325 2100 50  0000 L CNN
 	1    9325 2100
