File: LM358MicAmp/LM358MicAmp.kicad_pcb (KiCad board)
At the start: 2 copper layers, 13 parts, among them P1 CONN_01X02, P2 CONN_01X02, P3 CONN_01X02, P4 CONN_01X02, U1 LM358

Commit message: LM358 and LM317 bobs
Parts:
- removed P1, P2, P3, P4: CONN_01X02, Pin_Headers:Pin_Header_Straight_1x02_Pitch2.54mm
- added MIC: CONN_01X02, Pin_Headers:Pin_Header_Straight_1x02_Pitch2.54mm, F.Cu at (139.7, 94.0)
- added VCC: CONN_01X02, Pin_Headers:Pin_Header_Straight_1x02_Pitch2.54mm, F.Cu at (139.7, 101.6)
- added VOUT: CONN_01X02, Pin_Headers:Pin_Header_Straight_1x02_Pitch2.54mm, F.Cu at (139.7, 96.5)
- added VOUT_UC: CONN_01X02, Pin_Headers:Pin_Header_Straight_1x02_Pitch2.54mm, F.Cu at (139.7, 99.1)
- C1, CP2, R2, R3, R4, R5: moved to B.Cu
- moved U1 35.9 mm to (148.3, 94.5)
- moved R4 24.4 mm to (152.1, 101.3)
- moved R3 24.0 mm to (152.2, 98.8), turned to 180 degrees
- moved C1 14.5 mm to (152.2, 93.7), turned to 180 degrees
- moved CP2 14.0 mm to (145.5, 96.0), turned to 90 degrees
- moved CP1 13.6 mm to (145.5, 96.0), turned to 90 degrees
- moved R1 12.4 mm to (145.5, 101.9), turned to 90 degrees
- moved R5 11.8 mm to (152.1, 96.3), turned to 180 degrees
- moved R2 10.4 mm to (152.1, 104.1), turned to 180 degrees
Routing:
- net VCC: track 0.00 -> 24.0 mm, vias 0 -> 1
- net VOUT_UC: track 0.00 -> 14.3 mm
- net Net-(CP1-Pad2): track 0.00 -> 14.1 mm, vias 0 -> 2
- net Net-(R2-Pad1): track 0.00 -> 11.8 mm
- net MIC: track 0.00 -> 10.6 mm
- net Net-(R3-Pad2): track 0.00 -> 7.18 mm, vias 0 -> 2
- net VOUT: track 0.00 -> 4.47 mm
- net GND: track 0.00 -> 2.78 mm
- added copper zone on B.Cu, net GND
- added copper zone on F.Cu, net GND
Other:
- board outline added: 22.9 x 14 mm
- net class Default: trace_width 0.25 -> 0.2
- board text added: "Miracle CSP '17"
